Commit message: latest commit

File: fridge_bot/src/urdf/Fridge-bot.urdf (robot description, URDF)
Before this commit: robot Fridge-bot, 12 links, 11 joints
Links:
- added link world
Joints:
- added joint world_to_base_link=: type fixed, parent world, child base_link, origin xyz=0 0 1 rpy=0 0 0

File: fridge_bot/src/urdf/fridge_bot.urdf (robot description, URDF)
Before this commit: robot fridge_bot, 13 links, 12 joints
Links:
- link Back_gripper: mass 1.53802958602338 -> 0.167
- link front_halfgripper: mass 0.558596679661737 -> 0.06
Joints:
- joint joint3: limit lower=0 upper=6.28 effort=0 velocity=0 -> lower=0 upper=6.28 effort=1000 velocity=0.5; type revolute -> continuous
- joint joint7: limit lower=0 upper=6.28 effort=0 velocity=0 -> lower=0 upper=6.28 effort=1000 velocity=0.5; type revolute -> continuous
- joint world_to_base_link=: origin xyz=0 0 -.9 rpy=-1.57 0 0 -> xyz=0 0 0 rpy=0 0 0
