Commit message: fixed the robot orentation and updated the stl file

File: fridge_bot/src/urdf/fridge_bot.urdf (robot description, URDF)
Before this commit: robot fridge_bot, 13 links, 12 joints
Joints:
- joint world_to_base_link=: origin xyz=0 0 0 rpy=0 0 0 -> xyz=0 0 -.9 rpy=-1.57 0 0

Commit message: Latest Final Commit

File: fridge_bot/src/urdf/fridge_bot.urdf (robot description, URDF)
Before this commit: robot fridge_bot, 13 links, 12 joints
Joints:
- joint J10: limit lower=0 upper=6.28 effort=0 velocity=0 -> (none); type revolute -> fixed
